File: Anna ADD Pixie/Anna ADD Pixie.kicad_pcb (KiCad board)
At the start: 2 copper layers, 30.4 x 33.3 mm, 21 parts, among them J1 Conn_01x13_Pin, J2 Conn_01x02_Pin, J3 Conn_01x02_Pin, J4 Conn_01x01_Socket, J5 Conn_01x01_Socket, U1 MCP6002-xMC, U2 MCP6002-xMC

Commit message: Added INT module. Also updated ADD module with larger SJ holes.
Other:
- board text added: "{dblquote}Anna{dblquote} ADD Pixie 1.1 John Calhoun 2026"
- board text removed: "{dblquote}Anna{dblquote} ADD Pixie 1.0 John Calhoun 2026"
Changed lines of the file:
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@@
 			)
 		)
-		(pad "1" thru_hole rect
+		(pad "1" thru_hole circle
 			(at 0 0)
-			(size 1.7 1.7)
-			(drill 1)
+			(size 2.5 2.5)
+			(drill 1.5)
 			(layers "*.Cu" "*.Mask")
 			(remove_unused_layers no)
@@
 		(embedded_fonts no)
 		(model "${KICAD9_3DMODEL_DIR}/Connector_PinSocket_2.54mm.3dshapes/PinSocket_1x01_P2.54mm_Vertical.step"
+			(hide yes)
 			(offset
 				(xyz 0 0 0)
@@
 			)
 		)
-		(pad "1" thru_hole rect
+		(pad "1" thru_hole circle
 			(at 0 0)
-			(size 1.7 1.7)
-			(drill 1)
+			(size 2.5 2.5)
+			(drill 1.5)
 			(layers "*.Cu" "*.Mask")
 			(remove_unused_layers no)
@@
 		(embedded_fonts no)
 		(model "${KICAD9_3DMODEL_DIR}/Connector_PinSocket_2.54mm.3dshapes/PinSocket_1x01_P2.54mm_Vertical.step"
+			(hide yes)
 			(offset
 				(xyz 0 0 0)
@@
 		)
 	)
-	(gr_text "{dblquote}Anna{dblquote} ADD Pixie 1.0\nJohn Calhoun 2026"
+	(gr_text "{dblquote}Anna{dblquote} ADD Pixie 1.1\nJohn Calhoun 2026"
 		(at 154.3558 93.9292 0)
 		(layer "B.SilkS")
